File: mainboard/mainboard.kicad_sch (KiCad schematic)
At the start: 4 parts, among them J1 USB_B_Micro, U1 SX1276, U3 ATtiny85V-10M

Commit message: Updated mainboard, and schematics.
Parts:
- removed AE1: Antenna_Chip, symbol Device:Antenna_Chip
- removed U1: SX1276, Package_DFN_QFN:QFN-28-1EP_6x6mm_P0.65mm_EP4.8x4.8mm, symbol RF:SX1276
- removed U3: ATtiny85V-10M, Package_DFN_QFN:QFN-20-1EP_4x4mm_P0.5mm_EP2.6x2.6mm, symbol MCU_Microchip_ATtiny:ATtiny85V-10M
- added C1: 20pF, Capacitor_SMD:C_0201_0603Metric_Pad0.64x0.40mm_HandSolder, symbol Device:C
- added J2: Conn_Coaxial_Small, Connector_Coaxial:U.FL_Molex_MCRF_73412-0110_Vertical, symbol Connector:Conn_Coaxial_Small
- added R1: R, Resistor_SMD:R_0603_1608Metric, symbol Device:R
- added SC1: Solar_Cell, symbol Device:Solar_Cell
- added SW1, SW2: SW_Push, Button_Switch_SMD:SW_SPST_SKQG_WithoutStem, symbol Switch:SW_Push
- added U1: AMS1117-3.3, Package_TO_SOT_SMD:SOT-223-3_TabPin2, symbol Regulator_Linear:AMS1117-3.3
- added U2: STM32MP131AAEx, Package_BGA:LFBGA-289_14x14mm_Layout17x17_P0.8mm, symbol MCU_ST_STM32MP1:STM32MP131AAEx
- added U3: SX1276, Package_DFN_QFN:QFN-28-1EP_6x6mm_P0.65mm_EP4.8x4.8mm, symbol RF:SX1276
- added U4: nRF8001, Package_DFN_QFN:QFN-32-1EP_5x5mm_P0.5mm_EP3.45x3.45mm, symbol RF_Bluetooth:nRF8001
- added U5: BQ25570, Package_DFN_QFN:QFN-20-1EP_3.5x3.5mm_P0.5mm_EP2x2mm, symbol Battery_Management:BQ25570
- added Y1: Crystal_Small, Crystal:Crystal_SMD_MicroCrystal_CM9V-T1A-2Pin_1.6x1.0mm, symbol Device:Crystal_Small
Connections:
- net at J1.1 (VBUS): now also SW2.1
- net at J1.5 (GND): now also J2.2 (Ext), U1.1 (GND), U1.3 (VI), U3.15 (GND), U3.23 (GND), U3.26 (GND), U3.29 (GND)
- new net: J2.1 (In), U3.20 (RXTX/RF_MOD)
- new net: C1.2, R1.2, U3.5 (XTA), Y1.2
- new net: R1.1, U3.6 (XTB), Y1.1
- new net: SW2.2, U3.7 (~{RESET})
- new net: SW1.1, U1.2 (VO)
- new net: U5.1 (VSS), U5.15 (VSS), U5.17 (VSS), U5.21 (VSS), U5.9 (VSS)
- new net: U2.A1 (VSS), U2.A17 (VSS), U2.C8 (VSS), U2.D12 (VSS), U2.D3 (VSS), U2.E5 (VSS), U2.F13 (VSS), U2.F15 (VSS), U2.G10 (VSS), U2.G11 (VSS), U2.G7 (VSS), U2.G8 (VSS), U2.G9 (VSS), U2.H11 (VSS), U2.H14 (VSS), U2.H7 (VSS), U2.J11 (VSS), U2.J7 (VSS), U2.J9 (VSS), U2.K11 (VSS), U2.K3 (VSS), U2.K7 (VSS), U2.L10 (VSS), U2.L11 (VSS), U2.L7 (VSS), U2.L8 (VSS), U2.L9 (VSS), U2.M15 (VSS), U2.N4 (VSS), U2.P11 (VSS), U2.R5 (VSS), U2.R8 (VSS), U2.U1 (VSS), U2.U17 (VSS)
Other:
- moved on the sheet: J1
