File: portables/mainboard/_autosave-mainboard.kicad_sch (KiCad schematic)
At the start: 27 parts, among them J1 Conn_Coaxial, Q1 QM6006D, Q3 QM6015D, U1 SIM28ML, U3 BQ25570, U5 SX1279, U6 HDC1080, U8 MQ-6, U9 STM32WB15CCYx, Y1 TCXO-14, Y2 KC2520Z

Commit message: Worked on case, and still working on circuit.
Parts:
- added R4: 4.7kΩ, symbol Device:R
- added U2: PCF8584, symbol Interface_Expansion:PCF8584
- BT1: value Battery_Cell -> Na-Ion Cell (+5V,
Connections:
- net GND: now also Y2.2 (GND), R4.1
- net at C5.1, C8.1, L2.2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: now also Y2.4 (VCC), U2.20 (VDD)
- net at U1.9 (~{RESET}): no longer U9.E4 (PB2)
- net at Y2.1 (INH): now also U9.C6 (PB8), R4.2
- net at Y2.3 (CLK): now also U2.1 (CLK)
- now unconnected: U1.16 (TXD1/SDA), U1.17 (RXD1/SCL), U1.2 (TXD0), U1.3 (RXD0), U1.4 (TIMEMARK), U1.5 (EXTINT), U9.B4 (PB4), U9.E1 (PB1), U9.E2 (PB0)
- no-connect marks 23 -> 26
Other:
- moved on the sheet: U9, Y2
