File: portables/mainboard/mainboard.kicad_sch (KiCad schematic)
At the start: 28 parts, among them J1 Conn_Coaxial, Q1 QM6006D, Q3 QM6015D, U1 SIM28ML, U2 ATtiny85V-10S, U3 BQ25570, U4 PY32F002AW15U, U5 SX1279, U6 HDC1080, U7 ATtiny85V-10S, U8 MQ-6, Y1 TCXO-14

Commit message: Worked on case, and still working on circuit.
Parts:
- removed U2, U7: ATtiny85V-10S, Package_SO:SOIC-8_5.3x5.3mm_P1.27mm, symbol MCU_Microchip_ATtiny:ATtiny85V-10S
- removed U4: PY32F002AW15U, Package_DFN_QFN:WQFN-16-1EP_3x3mm_P0.5mm_EP1.75x1.75mm, symbol MCU_Puya:PY32F002AW15U
- added U2: PCF8584, symbol Interface_Expansion:PCF8584
- added U9: STM32WB15CCYx, Package_CSP:ST_WLCSP-49_3.3x3.38mm_Layout7x7_P0.4mm_Offcenter, symbol MCU_ST_STM32WB:STM32WB15CCYx
- added Y2: KC2520Z, Oscillator:Oscillator_SMD_Kyocera_KC2520Z-4Pin_2.5x2.0mm, symbol Oscillator:KC2520Z
Connections:
- net GND: now also U9.C3 (VSS), U9.D6 (VSS), U9.F5 (VSS)
- net at C5.1, C8.1, L2.2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: now also U2.20 (VDD), U9.C5 (VBAT)
- new net: U2.2 (SDA), U9.F7 (PA1)
- new net: U2.3 (SCL), U9.C4 (PA0)
- new net: U9.F4 (VSSRF), U9.G1 (VSSRF), U9.G3 (VSSRF)
Other:
- moved on the sheet: BT1, C1, C2, C3, C4, C5, C6, C7, C8, J1, L1, L2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
